Commit message: my changes

File: ca_description/urdf/create_base.urdf.xacro (robot description, xacro)
@@ -2,4 +2,8 @@
 <robot xmlns:xacro="http://ros.org/wiki/xacro">
   <xacro:property name="PI" value="3.1415926535897931" />
+    <property name="laserHeight" value="0.045" />
+    <property name="laserRadius" value="0.035" />
+    <property name="laserColor" value="red" />
+    <property name="laserMass" value="0.214" /> <!-- .5 lbs -->
   <xacro:macro name="create_wheel" params="prefix y_offset wheel_radius wheel_width">
     <link name="${prefix}_wheel_link">
@@ -28,5 +32,34 @@
       <axis xyz="0 1 0" />
     </joint>
-  </xacro:macro>
+   </xacro:macro>
+	<xacro:macro name="cylinder_inertia" params="m r h">
+	  <inertia
+			ixx="${m*(3*r*r+h*h)/12}" ixy = "0" ixz = "0"
+	    iyy="${m*(3*r*r+h*h)/12}" iyz = "0"
+	    izz="${m*r*r/2}"
+	  />
+	</xacro:macro>
+	<xacro:macro name="cylinder_link" params="name length radius mass color roll=0 pitch=${PI/2} yaw=${PI/2}">
+		<link name="${name}">
+		  <collision>
+		    <origin xyz="0 0 0" rpy="${roll} ${pitch} ${yaw}" />
+		    <geometry>
+		      <cylinder length="${length}" radius="${radius}"/>
+		    </geometry>
+		  </collision>
+		  <visual>
+		    <origin xyz="0 0 0" rpy="${roll} ${pitch} ${yaw}" />
+		    <geometry>
+		      <cylinder length="${length}" radius="${radius}"/>
+		    </geometry>
+		    <material name="${color}"/>
+		  </visual>
+		  <inertial>
+		    <origin xyz="0 0 0" rpy="${roll} ${pitch} ${yaw}" />
+		    <mass value="${mass}"/>
+		    <cylinder_inertia m="${mass}" r="${radius}" h="${length}"/>
+		  </inertial>
+		</link>
+	</xacro:macro>
   <xacro:macro name="create_base" params="diffdrive_update_rate:=40 wheel_separation wheel_radius:=0.036 wheel_width:=0.024 wheel_torque:=1.0 wheel_accel:=1.8 mass_kg:=3.5 base_diameter *mesh">
     <xacro:include filename="$(find ca_description)/urdf/create_base_gazebo.urdf.xacro" />
@@ -65,4 +98,5 @@
     </collision>
     </link>
+    <cylinder_link name="laser_link" length="${laserHeight}" radius="${laserRadius}" mass="${laserMass}" color="${laserColor}" pitch="0" yaw="0" />
     <link name="wall_sensor_link">
     <inertial>
@@ -104,4 +138,10 @@
       <parent link="base_footprint" />
       <child link="base_link" />
+    </joint>
+    <joint name="laser_joint" type="fixed">
+        <origin xyz="-0.0889 0 ${laserHeight*1.6+0.03175}" rpy="0 0 ${pi}"/>
+        <axis xyz="0 0 1"/>
+        <parent link="base_link"/>
+        <child link="laser_link"/>
     </joint>
     <joint name="base_wall_sensor_joint" type="fixed">

Commit message: added IMU

File: ca_description/urdf/create_base.urdf.xacro (robot description, xacro)
@@ -33,4 +33,11 @@
     </joint>
    </xacro:macro>
+	<macro name="box_inertia" params="m x y z">
+	  <inertia
+		  ixx="${m*(y*y+z*z)/12}" ixy = "0" ixz = "0"
+	    iyy="${m*(x*x+z*z)/12}" iyz = "0"
+	    izz="${m*(x*x+y*y)/12}"
+	  />
+	</macro>
 	<xacro:macro name="cylinder_inertia" params="m r h">
 	  <inertia
@@ -40,4 +47,26 @@
 	  />
 	</xacro:macro>
+	<macro name="box_link" params="name length width height mass color">
+		<link name="${name}">
+			<visual>
+				<origin xyz="0 0 0" rpy="0 0 0"/>
+				<geometry>
+					<box size="${length} ${width} ${height}"/>
+				</geometry>
+				<material name="${color}" />
+			</visual>
+			<collision>
+				<origin xyz="0 0 0" rpy="0 0 0" />
+				<geometry>
+					<box size="${length} ${width} ${height}"/>
+				</geometry>
+			</collision>
+			<inertial>
+				<origin xyz="0 0 0" rpy="0 0 0" />
+				<mass value="${mass}"/>
+				<box_inertia m="${mass}" x="${length}" y="${width}" z="${height}"/>
+			</inertial>
+		</link>
+	</macro>
 	<xacro:macro name="cylinder_link" params="name length radius mass color roll=0 pitch=${PI/2} yaw=${PI/2}">
 		<link name="${name}">
@@ -99,4 +128,5 @@
     </link>
     <cylinder_link name="laser_link" length="${laserHeight}" radius="${laserRadius}" mass="${laserMass}" color="${laserColor}" pitch="0" yaw="0" />
+    <box_link name="imu_link" length="0.03175" width="0.015875" height="0.0015875" mass="0.0283495" color="Yellow" />
     <link name="wall_sensor_link">
     <inertial>
@@ -144,4 +174,10 @@
         <parent link="base_link"/>
         <child link="laser_link"/>
+    </joint>
+    <joint name="imu_joint" type="fixed">
+        <origin xyz="0 0 ${0.0254+0.03175}" rpy="0 0 0"/>
+        <axis xyz="0 0 0"/>
+        <parent link="base_link"/>
+        <child link="imu_link"/>
     </joint>
     <joint name="base_wall_sensor_joint" type="fixed">
